File: docs/IRDocs/IR_Detector.kicad_sch (KiCad schematic)
At the start: 5 parts, among them J1 Raspberry_Pi_Zero_2_W, U1 TSOP4838, U2 TSOP4838

Commit message: Update detector schematics and BoM
Parts:
- added D1: LED_KRGB, symbol Device:LED_KRGB
Connections:
- net at C1.2, C2.2, J1.14 (GND)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: now also D1.1 (K)
- net at J1.32 (PWM0/GPIO12): now also D1.2 (RA)
- net at J1.33 (PWM1/GPIO13): now also D1.3 (GA)
- net at J1.35 (GPIO19/MISO1): now also D1.4 (BA)
Changed lines of the file:
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@@
+	)
+	(junction
+		(at 127 143.51)
+		(diameter 0)
+		(color 0 0 0 1)
 	)
 	(junction
@@
 	(wire
 		(pts
+			(xy 154.94 128.27) (xy 147.32 128.27)
+		)
+		(stroke
+			(width 0)
+			(type default)
+			(color 255 0 11 1)
+		)
+	)
+	(wire
+		(pts
+			(xy 100.33 152.4) (xy 154.94 152.4)
+		)
+		(stroke
+			(width 0)
+			(type default)
+			(color 255 0 11 1)
+		)
+	)
+	(wire
+		(pts
+			(xy 102.87 105.41) (xy 102.87 130.81)
+		)
+		(stroke
+			(width 0)
+			(type default)
+			(color 0 22 255 1)
+		)
+	)
+	(wire
+		(pts
+			(xy 153.67 149.86) (xy 97.79 149.86)
+		)
+		(stroke
+			(width 0)
+			(type default)
+		)
+	)
+	(wire
+		(pts
 			(xy 106.68 100.33) (xy 92.71 100.33)
 		)
@@
 	(wire
 		(pts
+			(xy 93.98 130.81) (xy 102.87 130.81)
+		)
+		(stroke
+			(width 0)
+			(type default)
+			(color 0 22 255 1)
+		)
+	)
+	(wire
+		(pts
 			(xy 185.42 88.9) (xy 182.88 88.9)
 		)
@@
 	(wire
 		(pts
+			(xy 154.94 152.4) (xy 154.94 128.27)
+		)
+		(stroke
+			(width 0)
+			(type default)
+			(color 255 0 11 1)
+		)
+	)
+	(wire
+		(pts
 			(xy 184.15 118.11) (xy 185.42 118.11)
 		)
@@
 	(wire
 		(pts
+			(xy 97.79 149.86) (xy 97.79 125.73)
+		)
+		(stroke
+			(width 0)
+			(type default)
+		)
+	)
+	(wire
+		(pts
 			(xy 182.88 123.19) (xy 195.58 123.19)
 		)
@@
 	(wire
 		(pts
+			(xy 80.01 143.51) (xy 127 143.51)
+		)
+		(stroke
+			(width 0)
+			(type default)
+			(color 0 0 0 1)
+		)
+	)
+	(wire
+		(pts
+			(xy 106.68 105.41) (xy 102.87 105.41)
+		)
+		(stroke
+			(width 0)
+			(type default)
+			(color 0 22 255 1)
+		)
+	)
+	(wire
+		(pts
 			(xy 184.15 125.73) (xy 184.15 128.27)
 		)
@@
 	(wire
 		(pts
+			(xy 83.82 125.73) (xy 80.01 125.73)
+		)
+		(stroke
+			(width 0)
+			(type default)
+			(color 0 0 0 1)
+		)
+	)
+	(wire
+		(pts
+			(xy 80.01 125.73) (xy 80.01 143.51)
+		)
+		(stroke
+			(width 0)
+			(type default)
+			(color 0 0 0 1)
+		)
+	)
+	(wire
+		(pts
 			(xy 97.79 54.61) (xy 191.77 54.61)
 		)
@@
 	(wire
 		(pts
+			(xy 100.33 120.65) (xy 100.33 152.4)
+		)
+		(stroke
+			(width 0)
+			(type default)
+			(color 255 0 11 1)
+		)
+	)
+	(wire
+		(pts
+			(xy 93.98 120.65) (xy 100.33 120.65)
+		)
+		(stroke
+			(width 0)
+			(type default)
+			(color 255 0 11 1)
+		)
+	)
+	(wire
+		(pts
+			(xy 147.32 130.81) (xy 153.67 130.81)
+		)
+		(stroke
+			(width 0)
+			(type default)
+		)
+	)
+	(wire
+		(pts
+			(xy 93.98 125.73) (xy 97.79 125.73)
+		)
+		(stroke
+			(width 0)
+			(type default)
+		)
+	)
+	(wire
+		(pts
 			(xy 184.15 128.27) (xy 190.5 128.27)
 		)
@@
 			(type default)
 			(color 0 64 255 1)
+		)
+	)
+	(wire
+		(pts
+			(xy 153.67 130.81) (xy 153.67 149.86)
+		)
+		(stroke
+			(width 0)
+			(type default)
 		)
 	)
@@
 					(unit 1)
 				)
+			)
+		)
+	)
+	(symbol
+		(lib_id "Device:LED_KRGB")
+		(at 88.9 125.73 0)
+		(unit 1)
+		(exclude_from_sim no)
+		(in_bom yes)
+		(on_board yes)
+		(dnp no)
+		(fields_autoplaced yes)
+		(property "Reference" "D1"
+			(at 88.9 111.76 0)
+			(effects
+				(font
+					(size 1.27 1.27)
+				)
+			)
+		)
+		(property "Value" "LED_KRGB"
+			(at 88.9 114.3 0)
+			(effects
+				(font
+					(size 1.27 1.27)
+				)
+			)
+		)
+		(property "Footprint" ""
+			(at 88.9 127 0)
+			(effects
+				(font
+					(size 1.27 1.27)
+				)
+				(hide yes)
+			)
+		)
+		(property "Datasheet" "~"
+			(at 88.9 127 0)
+			(effects
+				(font
+					(size 1.27 1.27)
+				)
+				(hide yes)
+			)
+		)
+		(property "Description" "RGB LED, cathode/red/green/blue"
+			(at 88.9 125.73 0)
+			(effects
+				(font
+					(size 1.27 1.27)
+				)
+				(hide yes)
+			)
+		)
+		(pin "2"
+		)
+		(pin "1"
+		)
+		(pin "4"
+		)
+		(pin "3"
+		)
+		(instances
+			(project ""
+				(path "/b27da0ba-d4c6-4bb1-a63c-5c17a72f8f7b"
+					(reference "D1")
+					(unit 1)
+				)

Commit message: doc update
Parts:
- added R1, R2: 100Ω, symbol Device:R_US
- added R3: 150Ω, symbol Device:R_US
Connections:
- net at D1.2 (RA): now also R3.1; no longer J1.32 (PWM0/GPIO12)
- net at D1.3 (GA): now also R2.1; no longer J1.33 (PWM1/GPIO13)
- net at D1.4 (BA): now also R1.2; no longer J1.35 (GPIO19/MISO1)
- new net: J1.32 (PWM0/GPIO12), R3.2
- new net: J1.35 (GPIO19/MISO1), R1.1
- new net: J1.33 (PWM1/GPIO13), R2.2
Changed lines of the file:
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@@
 	(wire
 		(pts
-			(xy 102.87 105.41) (xy 102.87 130.81)
+			(xy 99.06 105.41) (xy 99.06 107.95)
 		)
 		(stroke
@@
 	(wire
 		(pts
-			(xy 153.67 149.86) (xy 97.79 149.86)
+			(xy 153.67 149.86) (xy 125.73 149.86)
 		)
 		(stroke
@@
 	(wire
 		(pts
-			(xy 93.98 130.81) (xy 102.87 130.81)
+			(xy 93.98 130.81) (xy 99.06 130.81)
 		)
 		(stroke
@@
 	(wire
 		(pts
+			(xy 100.33 142.24) (xy 100.33 152.4)
+		)
+		(stroke
+			(width 0)
+			(type default)
+			(color 255 0 11 1)
+		)
+	)
+	(wire
+		(pts
 			(xy 121.92 63.5) (xy 185.42 63.5)
 		)
@@
 	(wire
 		(pts
-			(xy 106.68 105.41) (xy 102.87 105.41)
+			(xy 106.68 105.41) (xy 99.06 105.41)
 		)
 		(stroke
@@
 	(wire
 		(pts
+			(xy 99.06 115.57) (xy 99.06 130.81)
+		)
+		(stroke
+			(width 0)
+			(type default)
+			(color 0 22 255 1)
+		)
+	)
+	(wire
+		(pts
 			(xy 80.01 125.73) (xy 80.01 143.51)
 		)
@@
 	(wire
 		(pts
-			(xy 100.33 120.65) (xy 100.33 152.4)
+			(xy 118.11 149.86) (xy 97.79 149.86)
+		)
+		(stroke
+			(width 0)
+			(type default)
+		)
+	)
+	(wire
+		(pts
+			(xy 100.33 120.65) (xy 100.33 134.62)
 		)
 		(stroke
@@
 				(size 1.27 1.27)
 				(color 25 25 255 1)
+			)
+		)
+	)
+	(symbol
+		(lib_id "Device:R_US")
+		(at 100.33 138.43 0)
+		(unit 1)
+		(exclude_from_sim no)
+		(in_bom yes)
+		(on_board yes)
+		(dnp no)
+		(fields_autoplaced yes)
+		(property "Reference" "R3"
+			(at 102.87 137.1599 0)
+			(effects
+				(font
+					(size 1.27 1.27)
+				)
+				(justify left)
+			)
+		)
+		(property "Value" "150Ω"
+			(at 102.87 139.6999 0)
+			(effects
+				(font
+					(size 1.27 1.27)
+				)
+				(justify left)
+			)
+		)
+		(property "Footprint" ""
+			(at 101.346 138.684 90)
+			(effects
+				(font
+					(size 1.27 1.27)
+				)
+				(hide yes)
+			)
+		)
+		(property "Datasheet" "~"
+			(at 100.33 138.43 0)
+			(effects
+				(font
+					(size 1.27 1.27)
+				)
+				(hide yes)
+			)
+		)
+		(property "Description" "Resistor, US symbol"
+			(at 100.33 138.43 0)
+			(effects
+				(font
+					(size 1.27 1.27)
+				)
+				(hide yes)
+			)
+		)
+		(pin "1"
+		)
+		(pin "2"
+		)
+		(instances
+			(project "IR_Detector"
+				(path "/b27da0ba-d4c6-4bb1-a63c-5c17a72f8f7b"
+					(reference "R3")
+					(unit 1)
+				)
 			)
 		)
@@
 	)
 	(symbol
+		(lib_id "Device:R_US")
+		(at 99.06 111.76 0)
+		(unit 1)
+		(exclude_from_sim no)
+		(in_bom yes)
+		(on_board yes)
+		(dnp no)
+		(fields_autoplaced yes)
+		(property "Reference" "R1"
+			(at 101.6 110.4899 0)
+			(effects
+				(font
+					(size 1.27 1.27)
+				)
+				(justify left)
+			)
+		)
+		(property "Value" "100Ω"
+			(at 101.6 113.0299 0)
+			(effects
+				(font
+					(size 1.27 1.27)
+				)
+				(justify left)
+			)
+		)
+		(property "Footprint" ""
+			(at 100.076 112.014 90)
+			(effects
+				(font
+					(size 1.27 1.27)
+				)
+				(hide yes)
+			)
+		)
+		(property "Datasheet" "~"
+			(at 99.06 111.76 0)
+			(effects
+				(font
+					(size 1.27 1.27)
+				)
+				(hide yes)
+			)
+		)
+		(property "Description" "Resistor, US symbol"
+			(at 99.06 111.76 0)
+			(effects
+				(font
+					(size 1.27 1.27)
+				)
+				(hide yes)
+			)
+		)
+		(pin "1"
+		)
+		(pin "2"
+		)
+		(instances
+			(project ""
+				(path "/b27da0ba-d4c6-4bb1-a63c-5c17a72f8f7b"
+					(reference "R1")
+					(unit 1)
+				)
+			)
+		)
+	)
+	(symbol
 		(lib_id "Connector:Raspberry_Pi_2_3")
 		(at 127 110.49 0)
@@
 					(unit 1)
 				)
+			)
+		)
+	)
+	(symbol
+		(lib_id "Device:R_US")
+		(at 121.92 149.86 90)
+		(unit 1)
+		(exclude_from_sim no)
+		(in_bom yes)
+		(on_board yes)
+		(dnp no)
+		(fields_autoplaced yes)
+		(property "Reference" "R2"
+			(at 121.92 143.51 90)
+			(effects
+				(font
+					(size 1.27 1.27)
+				)
+			)
+		)
+		(property "Value" "100Ω"
+			(at 121.92 146.05 90)
+			(effects
+				(font
+					(size 1.27 1.27)
+				)
+			)
+		)
+		(property "Footprint" ""
+			(at 122.174 148.844 90)
+			(effects
+				(font
+					(size 1.27 1.27)
+				)
+				(hide yes)
+			)
+		)
+		(property "Datasheet" "~"
+			(at 121.92 149.86 0)
+			(effects
+				(font
+					(size 1.27 1.27)
+				)
+				(hide yes)
+			)
+		)
+		(property "Description" "Resistor, US symbol"
+			(at 121.92 149.86 0)
+			(effects
+				(font
+					(size 1.27 1.27)
+				)
+				(hide yes)
+			)
+		)
+		(pin "1"
+		)
+		(pin "2"
+		)
+		(instances
+			(project "IR_Detector"
+				(path "/b27da0ba-d4c6-4bb1-a63c-5c17a72f8f7b"
+					(reference "R2")
+					(unit 1)
+				)
